File: pcb/stackflex_core/stackflex_core.kicad_pcb (KiCad board)
At the start: 2 copper layers, 40 x 40 mm, 52 parts, among them IC1 ESP32-S3-MINI-1-N8, IC2 AP2112K-3.3TRG1, IC3 INA226AIDGSR, IC4 MAX17048G+T10, J1 USB_C_Receptacle_USB2.0_16P, J2 Conn_02x08_Counter_Clockwise, J3 Conn_02x08_Counter_Clockwise, J4 Conn_01x02_Socket, Q1 DMP2045U-7

Commit message: core 2025.1.1 and air quality 2025.1.0
Parts:
- removed R3, R4: 0, Resistor_SMD:R_0402_1005Metric
- added C10: 1uF, Capacitor_SMD:C_0402_1005Metric, F.Cu at (145.8, 107.4)
- added C11: 10uF, Capacitor_SMD:C_0402_1005Metric, F.Cu at (139.7, 108.5)
- added D4: red, stackflex_foots_lib:LEDC1005X55N, F.Cu at (139.4, 106.9)
- added G***: LOGO, stackflex_foots_lib:open_hw_logo_5mm_silk, B.Cu at (157.0, 112.5)
- added IC5: TP4054, stackflex_foots_lib:SOT95P280X100-5N, F.Cu at (143.0, 107.2)
- added JP1: SolderJumper_2_Open, Jumper:SolderJumper-2_P1.3mm_Open_TrianglePad1.0x1.5mm, B.Cu at (138.7, 110.5)
- R1: value 0 -> 1k
- R2: value 0 -> 2k
- R8: value .01 1% 250mW -> 33 mOhm 1% 250mW; footprint stackflex_foots_lib:RESC2013X45N -> Resistor_SMD:R_0805_2012Metric
- moved R1 9.91 mm to (137.2, 107.7)
- moved C3 4.89 mm to (135.4, 108.2), turned to 180 degrees
- moved R2 4.17 mm to (145.0, 104.9), turned to 0 degrees
- moved C7 3.06 mm to (136.4, 104.6), turned to 90 degrees
- moved C9 1.35 mm to (160.5, 108.2)
- moved R6 1.27 mm to (147.1, 107.4)
- moved R8 0.10 mm to (142.2, 103.3)
- turned S1 to 180 degrees
Connections:
- C3 pad 1: Net-(S1-N.O.) -> EN
- C8 pad 1: Net-(IC4-CELL) -> +BATT
- C9 pad 1: Net-(S2-N.O.) -> IO0
- IC4 pad 2: Net-(IC4-CELL) -> +BATT
- IC4 pad 3: Net-(IC4-CELL) -> +BATT
- J1 pad A6: Net-(J1-D+-PadA6) -> USB_D+
- J1 pad A7: Net-(J1-D--PadA7) -> USB_D-
- J1 pad B6: Net-(J1-D+-PadA6) -> USB_D+
- J1 pad B7: Net-(J1-D--PadA7) -> USB_D-
- R1 pad 1: Net-(J1-D--PadA7) -> Net-(JP1-A)
- R1 pad 2: USB_D- -> Net-(D4-A)
- R2 pad 1: Net-(J1-D+-PadA6) -> Net-(IC5-PROG)
- R2 pad 2: USB_D+ -> GND
- S1 pad 2: Net-(S1-N.O.) -> EN
- S2 pad 2: Net-(S2-N.O.) -> IO0
Routing:
- net +BATT: track 12.4 -> 30.4 mm, vias 1 -> 3
- net VBUS: track 15.9 -> 25.6 mm, vias 0 -> 1
- net EN: track 37.5 -> 46.4 mm, vias 2 -> 4
- net Net-(S1-N.O.): track 5.78 -> 0.00 mm
- net USB_D-: track 10.1 -> 15.8 mm
- net Net-(S2-N.O.): track 5.28 -> 0.00 mm
- net IO0: track 33.1 -> 38.1 mm
- net USB_D+: track 10.1 -> 15.0 mm
- net Net-(J1-D--PadA7): track 4.69 -> 0.00 mm
- net Net-(J1-D+-PadA6): track 4.11 -> 0.00 mm
- net Net-(JP1-A): track 0.00 -> 3.12 mm, vias 0 -> 1
- net 3V3_GPIO: track 95.9 -> 93.6 mm
- net GND: track 10.3 -> 12.6 mm, vias 28 -> 32
- net Net-(D4-K): track 0.00 -> 2.17 mm
- net Net-(IC4-CELL): track 1.89 -> 0.00 mm
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Other:
- board text added: "-"
- board text added: "3V3 GND IO3R IO4R NC NC SCLR SDAR CSR SCLKR MISOR MOSIR IO1R IO2R 3V3 GND"
- board text added: "CHRG LED"
- board text added: "GND 3V3 IO2L IO1L MOSIL MISOL SCLKL CSL SDAL SCLL NC NC IO4L IO3L GND 3V3"
- board text added: "JST-PH 2 mm"
- board text added: "L"
- board text added: "R"
- board text removed: "3V3 GND IO41 IO42 NC NC SCL1 SDA1 CS1 SCLK1 MISO1 MOSI1 IO34 IO48 3V3 GND"
- board text removed: "GND 3V3 IO1 IO2 MOSI0 MISO0 SCLK0 CS0 SDA0 SCL0 NC NC IO11 IO10 GND 3V3"
- board text removed: "JST-PH 2mm"
