File: pcb/stackflex_core/stackflex_core.kicad_sch (KiCad schematic)
At the start: 50 parts, among them IC1 ESP32-S3-MINI-1-N8, IC2 AP2112K-3.3TRG1, IC3 INA226AIDGSR, IC4 MAX17048G+T10, J1 USB_C_Receptacle_USB2.0_16P, J2 Conn_02x08_Counter_Clockwise, J3 Conn_02x08_Counter_Clockwise, J4 Conn_01x02_Socket, Q1 DMP2045U-7

Commit message: core 2025.1.1 and air quality 2025.1.0
Parts:
- removed R3, R4: 0, Resistor_SMD:R_0402_1005Metric, symbol Device:R_Small
- added C10: 1uF, Capacitor_SMD:C_0402_1005Metric, symbol Device:C_Small
- added C11: 10uF, Capacitor_SMD:C_0402_1005Metric, symbol Device:C_Small
- added D4: red, stackflex_foots_lib:LEDC1005X55N, symbol Device:LED_Small
- added IC5: TP4054, SOT95P280X100-5N, symbol stackflex_sym_lib:TP4054
- added JP1: SolderJumper_2_Open, Jumper:SolderJumper-2_P1.3mm_Open_TrianglePad1.0x1.5mm, symbol Jumper:SolderJumper_2_Open
- R1: value 0 -> 1k
- R2: value 0 -> 2k
- R8: value .01 1% 250mW -> 33 mOhm 1% 250mW; footprint stackflex_foots_lib:RESC2013X45N -> Resistor_SMD:R_0805_2012Metric
Connections:
- net +BATT: now also C8.1, IC4.2 (CELL), IC4.3 (VDD), C11.1, IC5.3 (BAT)
- net EN: now also C3.1, S1.2 (N.O.)
- net GND: now also R2.2, C10.2, C11.2, IC5.2 (GND)
- net IO0: now also C9.1, S2.2 (N.O.)
- net USB_D+: now also J1.A6 (D+), J1.B6 (D+); no longer R2.2
- net USB_D-: now also J1.A7 (D-), J1.B7 (D-); no longer R1.2
- net VBUS: now also C10.1, IC5.4 (VCC), JP1.2 (B)
- new net: JP1.1 (A), R1.1
- new net: D4.2 (A), R1.2
- new net: D4.1 (K), IC5.1 (~{CHRG})
- new net: IC5.5 (PROG), R2.1
Other:
- note added: "CSL"
- note added: "CSR"
- note added: "IO1L"
- note added: "IO1R"
- note added: "IO2L"
- note added: "IO2R"
- note added: "IO3L"
- note added: "IO3R"
- note added: "IO4L"
- note added: "IO4R"
- note added: "LiPo Charging"
- note added: "MISOL"
- note added: "MISOR"
- note added: "MOSIL"
- note added: "MOSIR"
- note added: "SCLKL"
- note added: "SCLKR"
- note added: "SCLL"
- note added: "SCLR"
- note added: "SDAL"
- note added: "SDAR"
- note added: "~1.5V @ 3.5mA"
- moved on the sheet: C6, J2, R5, S03, S4, S45, S46, S5
